File: spacehack_breakoutboard.sch (KiCad schematic (older format))
At the start: 2 parts, among them P1 HD44780 BUS, U1 BEAGLEBONEBLACK

Commit message: Added some more io ports
Parts:
- added P?: Inputs BUS, symbol CONN_20X2
- added P?: Nokia Bus, symbol CONN_20X2
Connections:
- net at U1.C1 (DGND): now also P?.1 (P1)
- net at U1.C3 (VDD_3V3EXP): now also P?.3 (P3)
- net at U1.B17 (GPIO0_27): now also P?.5 (P5)
- net at U1.B19 (EHRPWM2A): now also P?.7 (P7)
- net at U1.B21 (GPIO1_30): now also P?.9 (P9)
- net at U1.B23 (GPIO1_4): now also P?.11 (P11)
Changed lines of the file:
@@
 Sheet 1 1
 Title ""
-Date "5 mar 2014"
+Date "12 mar 2014"
 Rev ""
 Comp ""
@@
 Wire Wire Line
 	9400 4600 9100 4600
+$Comp
+L CONN_20X2 P?
+U 1 1 531E14AA
+P 1400 3700
+F 0 "P?" H 1400 4750 60  0000 C CNN
+F 1 "Inputs BUS" V 1400 3700 50  0000 C CNN
+F 2 "" H 1400 3700 60  0000 C CNN
+F 3 "" H 1400 3700 60  0000 C CNN
+	1    1400 3700
+	1    0    0    -1
+$EndComp
+Wire Wire Line
+	1000 2750 1000 2250
+Wire Wire Line
+	1000 2250 2800 2250
+Wire Wire Line
+	2800 2250 2800 2800
+Wire Wire Line
+	2800 2800 3050 2800
+Wire Wire Line
+	1000 2850 850  2850
+Wire Wire Line
+	850  2850 850  1950
+Wire Wire Line
+	850  1950 2700 1950
+Wire Wire Line
+	2700 1950 2700 2900
+Wire Wire Line
+	2700 2900 3050 2900
+$Comp
+L CONN_20X2 P?
+U 1 1 5320B02B
+P 1400 6100
+F 0 "P?" H 1400 7150 60  0000 C CNN
+F 1 "Nokia Bus" V 1400 6100 50  0000 C CNN
+F 2 "" H 1400 6100 60  0000 C CNN
+F 3 "" H 1400 6100 60  0000 C CNN
+	1    1400 6100
+	1    0    0    -1
+$EndComp
+Wire Wire Line
+	1000 2950 700  2950
+Wire Wire Line
+	700  2950 700  1800
+Wire Wire Line
+	700  1800 5650 1800
+Wire Wire Line
+	5650 1800 5650 3600
+Wire Wire Line
+	5650 3600 6250 3600
+Wire Wire Line
+	1000 3050 600  3050
+Wire Wire Line
+	600  3050 600  4800
+Wire Wire Line
+	600  4800 2650 4800
+Wire Wire Line
+	2650 4800 2650 5300
+Wire Wire Line
+	2650 5300 5650 5300
+Wire Wire Line
+	5650 5300 5650 3700
+Wire Wire Line
+	5650 3700 6250 3700
+Wire Wire Line
+	1000 3150 750  3150
+Wire Wire Line
+	750  3150 750  4950
+Wire Wire Line
+	750  4950 2500 4950
+Wire Wire Line
+	2500 4950 2500 5450
+Wire Wire Line
+	2500 5450 5800 5450
+Wire Wire Line
+	5800 5450 5800 3800
+Wire Wire Line
+	5800 3800 6250 3800
+Wire Wire Line
+	1000 3250 900  3250
+Wire Wire Line
+	900  3250 900  5050
+Wire Wire Line
+	900  5050 2400 5050
+Wire Wire Line
+	2400 5050 2400 5600
+Wire Wire Line
+	2400 5600 5900 5600
+Wire Wire Line
+	5900 5600 5900 3900
+Wire Wire Line
+	5900 3900 6250 3900
 $EndSCHEMATC
