File: spacehack_breakoutboard.kicad_pcb (KiCad board)
At the start: 2 copper layers, 208.3 x 132.1 mm, 2 parts, among them P1 HD44780 BUS, U1 BEAGLEBONEBLACK

Commit message: Really rough layout
Parts:
- moved P1 21.6 mm to (200.7, 170.2)
- moved U1 0.42 mm to (182.0, 117.0)
Routing:
- net N-0000032: track 39.6 -> 166.2 mm, vias 0 -> 2
- net N-0000037: track 51.8 -> 143.7 mm, vias 1 -> 2
- net GND: track 102.5 -> 168.2 mm
- net N-000004: track 36.9 -> 95.6 mm, vias 0 -> 2
- net +5V: track 111.8 -> 167.4 mm
- net N-0000030: track 123.0 -> 164.3 mm, vias 1 -> 2
- net N-0000035: track 72.5 -> 112.9 mm
- net +3.3V: track 111.8 -> 152.3 mm, vias 2 -> 0
- net (no net): track 36.1 -> 0.00 mm
- net N-0000026: track 89.4 -> 120.7 mm
- net N-0000024: track 8.78 -> 30.5 mm
- net N-0000033: track 9.83 -> 31.5 mm
- net N-0000021: track 60.5 -> 46.2 mm, vias 1 -> 0
